Commit message: Twist Inputs & Odometry feedbacks now work with the new Driver!

File: omni_bot/description/bot.xacro (robot description, xacro)
@@ -12,4 +12,6 @@
   <xacro:property name="rod_width" value="0.02" /> <!-- m -->
   <xacro:property name="chassis_offset" value="0.01" /> <!-- m -->
+  <xacro:property name="encoder_radius" value="0.05" /> <!-- m -->
+  <xacro:property name="encoder_scale" value="${100/152}" /> <!-- m -->
   <!-- Derived Vars -->
   <xacro:property name="base_height" value="${1.732 * base_side_length / 2}" /> <!-- m -->
@@ -61,3 +63,10 @@
     <origin xyz="${((2 * base_height / 3) - (1.732 * corner_side_length / 2) - (rod_width / 2) - shaft_length)* cos(pi/6)} -${((2 * base_height / 3) - (1.732 * corner_side_length / 2) - (rod_width / 2) - shaft_length) * sin(pi/6)} ${wheel_radius}" rpy="${pi/2} 0.0 -${pi/6 + pi/2}"/>
   </xacro:wheel>
+  <!-- Encoders -->
+  <xacro:encoder pos="X" parent="base_link" scale="${encoder_scale}">
+    <origin xyz="0.0 0.08 ${encoder_radius}" rpy="-${pi/2} 0.0 0.0"/>  <!-- 0.09 is experimental value -->
+  </xacro:encoder>
+  <xacro:encoder pos="Y" parent="base_link" scale="${encoder_scale}">
+    <origin xyz="-0.04 -0.04 ${encoder_radius}" rpy="0.0 -${pi/2} 0.0"/> <!-- 0.042 and 0.03 are experimental values -->
+  </xacro:encoder>
 </robot>

File: omni_bot/description/omni_bot.urdf.xacro (robot description, xacro)
@@ -4,6 +4,6 @@
   <xacro:include filename="bot.xacro"/>
   <!-- Gazebo Parameters -->
-  <xacro:include filename="gazebo_params_ros2.xacro"/>
+  <!-- <xacro:include filename="gazebo_params_ros2.xacro"/> -->
   <!-- ROS2 Control -->
-  <xacro:include filename="ros2_control.xacro"/>
+  <!-- <xacro:include filename="ros2_control.xacro"/> -->
 </robot>

File: omni_bot/description/wheels.xacro (robot description, xacro)
@@ -112,3 +112,28 @@
     <xacro:insert_wheel parent="${pos}_wheel_link" reflect="1" prefix="${pos}" suffix="2" />
   </xacro:macro>
+  <!-- Encoder Wheel Spawn Macro -->
+  <xacro:macro name="encoder" params="pos parent *origin scale">
+    <joint name="${pos}_encoder_joint" type="continuous">
+      <xacro:insert_block name="origin"/>
+      <parent link="${parent}"/>
+      <child link="${pos}_encoder_link"/>
+      <axis xyz="0 0 1"/>
+    </joint>
+    <link name="${pos}_encoder_link">
+      <visual>
+        <origin rpy="${pi/2} 0.0 0.0"/>
+        <geometry>
+          <mesh filename="file://$(find omni_bot)/description/meshes/omni_wheel_152mm.stl" scale="${scale} ${scale} ${scale}"/>
+        </geometry>
+        <material name="light_gray">
+          <color rgba="0.75 0.75 0.75 1.0"/>
+        </material>
+      </visual>
+      <collision>
+        <geometry>
+          <cylinder radius="0.073" length="0.03"/>  <!-- Experimental values -->
+        </geometry>
+      </collision>
+    </link>
+  </xacro:macro>
 </robot>

Commit message: Bot works, just waiting on getting the RPi to get a github acc to push...

File: omni_bot/description/bot.xacro (robot description, xacro)
@@ -2,5 +2,5 @@
 <robot xmlns:xacro="http://www.ros.org/wiki/xacro">
   <!-- Includes -->
-  <xacro:include filename="wheels.xacro"/>
+  <xacro:include filename="wheels.xacro" />
   <!-- Variables -->
   <xacro:property name="base_mass" value="3.214" /> <!-- kg -->
@@ -16,22 +16,29 @@
   <!-- Derived Vars -->
   <xacro:property name="base_height" value="${1.732 * base_side_length / 2}" /> <!-- m -->
-  <!-- Body -->
-  <link name="base_link"/>
+  <!-- Base Link -->
   <joint name="base_joint" type="fixed">
-    <parent link="base_link"/>
-    <child link="body_link"/>
+    <parent link="base_link" />
+    <child link="body_link" />
   </joint>
+  <link name="base_link" />
+  <!-- Base Footprint -->
+  <joint name="base_footprint_joint" type="fixed">
+    <parent link="base_link" />
+    <child link="base_footprint" />
+  </joint>
+  <link name="base_footprint" />
+  <!-- Base -->
   <link name="body_link">
     <visual>
-      <origin xyz="0.0 -${base_height/3} ${base_clearance - chassis_offset}" rpy="0.0 0.0 ${pi/6}"/>
+      <origin xyz="0.0 -${base_height/3} ${base_clearance - chassis_offset}" rpy="0.0 0.0 ${pi/6}" />
       <geometry>
         <mesh filename="file://$(find omni_bot)/description/meshes/chassis.stl" />
       </geometry>
       <material name="light_gray">
-        <color rgba="0.75 0.75 0.75 1.0"/>
+        <color rgba="0.75 0.75 0.75 1.0" />
       </material>
     </visual>
     <collision>
-      <origin xyz="0.0 -${base_height/3} ${base_clearance}" rpy="0.0 0.0 ${pi/6}"/>
+      <origin xyz="0.0 -${base_height/3} ${base_clearance}" rpy="0.0 0.0 ${pi/6}" />
       <geometry>
         <mesh filename="file://$(find omni_bot)/description/meshes/bot_base.stl" />
@@ -40,12 +47,12 @@
     <inertial>
       <!-- <origin xyz="0.0 ${-base_height/3} ${base_clearance}" rpy="0.0 0.0 ${pi/6}"/> -->
-      <origin xyz="0.0 0.0 ${base_clearance}" rpy="0.0 0.0 0.0"/>
-      <mass value="${base_mass}"/>
+      <origin xyz="0.0 0.0 ${base_clearance}" rpy="0.0 0.0 0.0" />
+      <mass value="${base_mass}" />
       <inertia ixx="0.1798003"
-                ixy="0.0024346"
-                ixz="-0.0001306"
-                iyy="0.1827598"
-                iyz="-0.0002425"
-                izz="0.3538762"/>
+        ixy="0.0024346"
+        ixz="-0.0001306"
+        iyy="0.1827598"
+        iyz="-0.0002425"
+        izz="0.3538762" />
     </inertial>
   </link>
@@ -55,18 +62,57 @@
   <!-- Wheels -->
   <xacro:wheel pos="front" parent="base_link">
-    <origin xyz="0.0 ${2 * base_height / 3 - (1.732 * corner_side_length / 2) - (rod_width / 2) - shaft_length} ${wheel_radius}" rpy="${pi/2} 0.0 0.0"/>
+    <origin
+      xyz="0.0 ${2 * base_height / 3 - (1.732 * corner_side_length / 2) - (rod_width / 2) - shaft_length} ${wheel_radius}"
+      rpy="${pi/2} 0.0 0.0" />
   </xacro:wheel>
   <xacro:wheel pos="left" parent="base_link">
-    <origin xyz="-${((2 * base_height / 3) - (1.732 * corner_side_length / 2) - (rod_width / 2) - shaft_length)* cos(pi/6)} -${((2 * base_height / 3) - (1.732 * corner_side_length / 2) - (rod_width / 2) - shaft_length) * sin(pi/6)} ${wheel_radius}" rpy="${pi/2} 0.0 ${pi/6 + pi/2}"/>
+    <origin
+      xyz="-${((2 * base_height / 3) - (1.732 * corner_side_length / 2) - (rod_width / 2) - shaft_length)* cos(pi/6)} -${((2 * base_height / 3) - (1.732 * corner_side_length / 2) - (rod_width / 2) - shaft_length) * sin(pi/6)} ${wheel_radius}"
+      rpy="${pi/2} 0.0 ${pi/6 + pi/2}" />
   </xacro:wheel>
   <xacro:wheel pos="right" parent="base_link">
-    <origin xyz="${((2 * base_height / 3) - (1.732 * corner_side_length / 2) - (rod_width / 2) - shaft_length)* cos(pi/6)} -${((2 * base_height / 3) - (1.732 * corner_side_length / 2) - (rod_width / 2) - shaft_length) * sin(pi/6)} ${wheel_radius}" rpy="${pi/2} 0.0 -${pi/6 + pi/2}"/>
+    <origin
+      xyz="${((2 * base_height / 3) - (1.732 * corner_side_length / 2) - (rod_width / 2) - shaft_length)* cos(pi/6)} -${((2 * base_height / 3) - (1.732 * corner_side_length / 2) - (rod_width / 2) - shaft_length) * sin(pi/6)} ${wheel_radius}"
+      rpy="${pi/2} 0.0 -${pi/6 + pi/2}" />
   </xacro:wheel>
   <!-- Encoders -->
   <xacro:encoder pos="X" parent="base_link" scale="${encoder_scale}">
-    <origin xyz="0.0 0.08 ${encoder_radius}" rpy="-${pi/2} 0.0 0.0"/>  <!-- 0.09 is experimental value -->
+    <origin xyz="0.0 0.08 ${encoder_radius}" rpy="-${pi/2} 0.0 0.0" />  <!-- 0.09 is experimental
+    value -->
   </xacro:encoder>
   <xacro:encoder pos="Y" parent="base_link" scale="${encoder_scale}">
-    <origin xyz="-0.04 -0.04 ${encoder_radius}" rpy="0.0 -${pi/2} 0.0"/> <!-- 0.042 and 0.03 are experimental values -->
+    <origin xyz="-0.04 -0.04 ${encoder_radius}" rpy="0.0 -${pi/2} 0.0" /> <!-- 0.042 and 0.03 are
+    experimental values -->
   </xacro:encoder>
+  <!-- Lidar -->
+  <joint name="lidar_joint" type="continuous">
+    <parent link="base_link" />
+    <child link="lidar_link" />
+    <origin xyz="0.0 0.0 0.15" rpy="0.0 0.0 ${pi}" />
+  </joint>
+  <link name="lidar_link">
+    <visual>
+      <origin xyz="0.0 0.0 0.0" rpy="0.0 0.0 0.0" />
+      <geometry>
+        <mesh filename="file://$(find omni_bot)/description/meshes/Scanner.stl" />
+      </geometry>
+      <material name="dark_gray">
+        <color rgba="0.25 0.25 0.25 1.0" />
+      </material>
+    </visual>
+    <collision>
+      <origin xyz="0.0 0.0 0.0" rpy="0.0 0.0 0.0" />
+      <geometry>
+        <mesh filename="file://$(find omni_bot)/description/meshes/Scanner.stl" />
+      </geometry>
+    </collision>
+    <inertial>
+      <origin xyz="0.0 0.0 0.0" rpy="0.0 0.0 0.0" />
+      <mass value="0.1" />
+      <inertia ixx="0.0001" ixy="0.0" ixz="0.0" iyy="0.0001" iyz="0.0" izz="0.0001" />
+    </inertial>
+  </link>
+  <gazebo reference="lidar_link">
+    <material>Gazebo/Black</material>
+  </gazebo>
 </robot>

File: omni_bot/description/omni_bot.urdf.xacro (robot description, xacro)
@@ -1,9 +1,5 @@
 <?xml version="1.0"?>
 <robot xmlns:xacro="http://www.ros.org/wiki/xacro" name="omni_bot">
-  <!-- Bot Description -->
+  <!-- Bot Description URDF -->
   <xacro:include filename="bot.xacro"/>
-  <!-- Gazebo Parameters -->
-  <!-- <xacro:include filename="gazebo_params_ros2.xacro"/> -->
-  <!-- ROS2 Control -->
-  <!-- <xacro:include filename="ros2_control.xacro"/> -->
 </robot>

File: omni_bot/description/wheels.xacro (robot description, xacro)
@@ -6,5 +6,5 @@
   <!-- Roller Spawn Macro -->
   <xacro:macro name="insert_roller" params="parent theta prefix suffix">
-    <joint name="${prefix}_roller_${suffix}_joint" type="continuous">
+    <joint name="${prefix}_roller_${suffix}_joint" type="fixed">
       <origin xyz="${distance_to_roller_center*cos(theta)} ${distance_to_roller_center*sin(theta)} 0.0" rpy="0.0 0.0 ${theta-pi/2}"/>
       <parent link="${parent}"/>
@@ -96,5 +96,5 @@
   <!-- Wheel Spawn Macro -->
   <xacro:macro name="wheel" params="pos parent *origin">
-    <joint name="${pos}_wheel_joint" type="continuous">
+    <joint name="${pos}_wheel_joint" type="fixed">
       <xacro:insert_block name="origin"/>
       <parent link="${parent}"/>

Commit message: Added mapping stuff

File: omni_bot/description/bot.xacro (robot description, xacro)
@@ -26,4 +26,5 @@
     <parent link="base_link" />
     <child link="base_footprint" />
+    <origin rpy="0.0 0.0 ${pi/2}"/>
   </joint>
   <link name="base_footprint" />
@@ -86,6 +87,6 @@
   </xacro:encoder>
   <!-- Lidar -->
-  <joint name="lidar_joint" type="continuous">
-    <parent link="base_link" />
+  <joint name="lidar_joint" type="fixed">
+    <parent link="base_footprint" />
     <child link="lidar_link" />
     <origin xyz="0.0 0.0 0.15" rpy="0.0 0.0 ${pi}" />
