Commit message: QoL: Differentiated packages targetting Real Bot from Sim.

File: omni_bot_sim/description/bot.xacro (robot description, xacro)
@@ -34,5 +34,5 @@
       <origin xyz="0.0 -${base_height/3} ${base_clearance - chassis_offset}" rpy="0.0 0.0 ${pi/6}" />
       <geometry>
-        <mesh filename="file://$(find omni_bot)/description/meshes/chassis.stl" />
+        <mesh filename="file://$(find omni_bot_sim)/description/meshes/chassis.stl" />
       </geometry>
       <material name="light_gray">
@@ -43,5 +43,5 @@
       <origin xyz="0.0 -${base_height/3} ${base_clearance}" rpy="0.0 0.0 ${pi/6}" />
       <geometry>
-        <mesh filename="file://$(find omni_bot)/description/meshes/bot_base.stl" />
+        <mesh filename="file://$(find omni_bot_sim)/description/meshes/bot_base.stl" />
       </geometry>
     </collision>
@@ -96,5 +96,5 @@
       <origin xyz="0.0 0.0 0.0" rpy="0.0 0.0 0.0" />
       <geometry>
-        <mesh filename="file://$(find omni_bot)/description/meshes/Scanner.stl" />
+        <mesh filename="file://$(find omni_bot_sim)/description/meshes/Scanner.stl" />
       </geometry>
       <material name="dark_gray">
@@ -105,5 +105,5 @@
       <origin xyz="0.0 0.0 0.0" rpy="0.0 0.0 0.0" />
       <geometry>
-        <mesh filename="file://$(find omni_bot)/description/meshes/Scanner.stl" />
+        <mesh filename="file://$(find omni_bot_sim)/description/meshes/Scanner.stl" />
       </geometry>
     </collision>

File: omni_bot_sim/description/wheels.xacro (robot description, xacro)
@@ -16,5 +16,5 @@
       <visual>
         <geometry>
-            <mesh filename="file://$(find omni_bot)/description/meshes/omni_wheel_roller.stl"/>
+            <mesh filename="file://$(find omni_bot_sim)/description/meshes/omni_wheel_roller.stl"/>
         </geometry>
         <material name="black">
@@ -53,5 +53,5 @@
         <origin rpy="${pi/2} 0.0 ${2*pi/28}"/>
         <geometry>
-          <mesh filename="file://$(find omni_bot)/description/meshes/omni_wheel_plate.stl"/>
+          <mesh filename="file://$(find omni_bot_sim)/description/meshes/omni_wheel_plate.stl"/>
         </geometry>
         <material name="gray">
@@ -62,5 +62,5 @@
                 <origin rpy="${pi/2} 0.0 ${2*pi/28}"/>
                 <geometry>
-                    <mesh filename="file://$(find omni_bot)/description/meshes/omni_wheel_plate.stl"/>
+                    <mesh filename="file://$(find omni_bot_sim)/description/meshes/omni_wheel_plate.stl"/>
                 </geometry>
       </collision> -->
@@ -124,5 +124,5 @@
         <origin rpy="${pi/2} 0.0 0.0"/>
         <geometry>
-          <mesh filename="file://$(find omni_bot)/description/meshes/omni_wheel_152mm.stl" scale="${scale} ${scale} ${scale}"/>
+          <mesh filename="file://$(find omni_bot_sim)/description/meshes/omni_wheel_152mm.stl" scale="${scale} ${scale} ${scale}"/>
         </geometry>
         <material name="light_gray">
