Commit message: QoL Pt.2: Yet another change to simplify stuff.

File: omni_bot_description/description/bot.xacro (robot description, xacro)
@@ -34,5 +34,5 @@
       <origin xyz="0.0 -${base_height/3} ${base_clearance - chassis_offset}" rpy="0.0 0.0 ${pi/6}" />
       <geometry>
-        <mesh filename="file://$(find omni_bot_sim)/description/meshes/chassis.stl" />
+        <mesh filename="file://$(find omni_bot_description)/description/meshes/chassis.stl" />
       </geometry>
       <material name="light_gray">
@@ -43,5 +43,5 @@
       <origin xyz="0.0 -${base_height/3} ${base_clearance}" rpy="0.0 0.0 ${pi/6}" />
       <geometry>
-        <mesh filename="file://$(find omni_bot_sim)/description/meshes/bot_base.stl" />
+        <mesh filename="file://$(find omni_bot_description)/description/meshes/bot_base.stl" />
       </geometry>
     </collision>
@@ -96,5 +96,5 @@
       <origin xyz="0.0 0.0 0.0" rpy="0.0 0.0 0.0" />
       <geometry>
-        <mesh filename="file://$(find omni_bot_sim)/description/meshes/Scanner.stl" />
+        <mesh filename="file://$(find omni_bot_description)/description/meshes/Scanner.stl" />
       </geometry>
       <material name="dark_gray">
@@ -105,5 +105,5 @@
       <origin xyz="0.0 0.0 0.0" rpy="0.0 0.0 0.0" />
       <geometry>
-        <mesh filename="file://$(find omni_bot_sim)/description/meshes/Scanner.stl" />
+        <mesh filename="file://$(find omni_bot_description)/description/meshes/Scanner.stl" />
       </geometry>
     </collision>

File: omni_bot_description/description/wheels.xacro (robot description, xacro)
@@ -16,5 +16,5 @@
       <visual>
         <geometry>
-            <mesh filename="file://$(find omni_bot_sim)/description/meshes/omni_wheel_roller.stl"/>
+            <mesh filename="file://$(find omni_bot_description)/description/meshes/omni_wheel_roller.stl"/>
         </geometry>
         <material name="black">
@@ -53,5 +53,5 @@
         <origin rpy="${pi/2} 0.0 ${2*pi/28}"/>
         <geometry>
-          <mesh filename="file://$(find omni_bot_sim)/description/meshes/omni_wheel_plate.stl"/>
+          <mesh filename="file://$(find omni_bot_description)/description/meshes/omni_wheel_plate.stl"/>
         </geometry>
         <material name="gray">
@@ -62,5 +62,5 @@
                 <origin rpy="${pi/2} 0.0 ${2*pi/28}"/>
                 <geometry>
-                    <mesh filename="file://$(find omni_bot_sim)/description/meshes/omni_wheel_plate.stl"/>
+                    <mesh filename="file://$(find omni_bot_description)/description/meshes/omni_wheel_plate.stl"/>
                 </geometry>
       </collision> -->
@@ -124,5 +124,5 @@
         <origin rpy="${pi/2} 0.0 0.0"/>
         <geometry>
-          <mesh filename="file://$(find omni_bot_sim)/description/meshes/omni_wheel_152mm.stl" scale="${scale} ${scale} ${scale}"/>
+          <mesh filename="file://$(find omni_bot_description)/description/meshes/omni_wheel_152mm.stl" scale="${scale} ${scale} ${scale}"/>
         </geometry>
         <material name="light_gray">

Commit message: Cleared up some redundancies from desription & added an IMU sensor.

File: omni_bot_description/description/bot.xacro (robot description, xacro)
@@ -8,5 +8,5 @@
   <xacro:property name="base_clearance" value="0.048" /> <!-- m -->
   <xacro:property name="wheel_radius" value="0.076" /> <!-- m -->
-  <xacro:property name="shaft_length" value="0.05" /> <!-- m -->
+  <xacro:property name="shaft_length" value="0.055" /> <!-- m -->
   <xacro:property name="corner_side_length" value="0.15" /> <!-- m -->
   <xacro:property name="rod_width" value="0.02" /> <!-- m -->
@@ -22,9 +22,8 @@
   </joint>
   <link name="base_link" />
-  <!-- Base Footprint -->
+  <!-- Base Footprint (Required by some controllers) -->
   <joint name="base_footprint_joint" type="fixed">
     <parent link="base_link" />
     <child link="base_footprint" />
-    <origin rpy="0.0 0.0 ${pi/2}"/>
   </joint>
   <link name="base_footprint" />
@@ -35,4 +34,5 @@
       <geometry>
         <mesh filename="file://$(find omni_bot_description)/description/meshes/chassis.stl" />
+        <!-- <mesh filename="meshes/chassis.stl" /> -->
       </geometry>
       <material name="light_gray">
@@ -41,7 +41,8 @@
     </visual>
     <collision>
-      <origin xyz="0.0 -${base_height/3} ${base_clearance}" rpy="0.0 0.0 ${pi/6}" />
+      <origin xyz="0.0 -${base_height/3} ${base_clearance - chassis_offset}" rpy="0.0 0.0 ${pi/6}" />
       <geometry>
-        <mesh filename="file://$(find omni_bot_description)/description/meshes/bot_base.stl" />
+        <mesh filename="file://$(find omni_bot_description)/description/meshes/chassis.stl" />
+        <!-- <mesh filename="meshes/chassis.stl" /> -->
       </geometry>
     </collision>
@@ -86,4 +87,26 @@
     experimental values -->
   </xacro:encoder>
+  <!-- IMU -->
+  <joint name="imu_joint" type="fixed">
+    <parent link="base_footprint" />
+    <child link="imu_link" />
+    <origin xyz="0.0 0.0 ${base_clearance + 0.1}" rpy="0.0 0.0 0.0" />
+  </joint>
+  <link name="imu_link">
+    <visual>
+      <geometry>
+        <mesh filename="file://$(find omni_bot_description)/description/meshes/MPU_6050.stl" scale="0.001 0.001 0.001"/>
+        <!-- <mesh filename="meshes/MPU_6050.stl" scale="0.001 0.001 0.001"/> -->
+      </geometry>
+      <material name="dark_gray">
+        <color rgba="0.25 0.25 0.25 1.0" />
+      </material>
+    </visual>
+    <collision>
+      <geometry>
+        <box size="0.02 0.015 0.003"/>
+      </geometry>
+    </collision>
+  </link>
   <!-- Lidar -->
   <joint name="lidar_joint" type="fixed">
@@ -94,7 +117,7 @@
   <link name="lidar_link">
     <visual>
-      <origin xyz="0.0 0.0 0.0" rpy="0.0 0.0 0.0" />
       <geometry>
         <mesh filename="file://$(find omni_bot_description)/description/meshes/Scanner.stl" />
+        <!-- <mesh filename="meshes/Scanner.stl" /> -->
       </geometry>
       <material name="dark_gray">
@@ -103,11 +126,10 @@
     </visual>
     <collision>
-      <origin xyz="0.0 0.0 0.0" rpy="0.0 0.0 0.0" />
       <geometry>
         <mesh filename="file://$(find omni_bot_description)/description/meshes/Scanner.stl" />
+        <!-- <mesh filename="meshes/Scanner.stl" /> -->
       </geometry>
     </collision>
     <inertial>
-      <origin xyz="0.0 0.0 0.0" rpy="0.0 0.0 0.0" />
       <mass value="0.1" />
       <inertia ixx="0.0001" ixy="0.0" ixz="0.0" iyy="0.0001" iyz="0.0" izz="0.0001" />

File: omni_bot_description/description/wheels.xacro (robot description, xacro)
@@ -1,97 +1,4 @@
 <?xml version="1.0"?>
 <robot xmlns:xacro="http://www.ros.org/wiki/xacro">
-  <!-- Variables -->
-  <xacro:property name="distance_to_roller_center" value="0.065"/>
-  <xacro:property name="inter_wheel_gap" value="0.02"/>
-  <!-- Roller Spawn Macro -->
-  <xacro:macro name="insert_roller" params="parent theta prefix suffix">
-    <joint name="${prefix}_roller_${suffix}_joint" type="fixed">
-      <origin xyz="${distance_to_roller_center*cos(theta)} ${distance_to_roller_center*sin(theta)} 0.0" rpy="0.0 0.0 ${theta-pi/2}"/>
-      <parent link="${parent}"/>
-      <child link="${prefix}_roller_${suffix}_link"/>
-      <axis xyz="1.0 0.0 0.0"/>
-      <!-- <dynamics friction="0.1"/> -->
-    </joint>
-    <link name="${prefix}_roller_${suffix}_link">
-      <visual>
-        <geometry>
-            <mesh filename="file://$(find omni_bot_description)/description/meshes/omni_wheel_roller.stl"/>
-        </geometry>
-        <material name="black">
-            <color rgba="0.0 0.0 0.0 1.0"/>
-        </material>
-      </visual>
-      <collision>
-          <origin rpy="0.0 ${pi/2} 0.0"/>
-          <geometry>
-              <cylinder radius="0.0095" length="0.018"/>  <!-- CAD values -->
-          </geometry>
-      </collision>
-      <inertial>
-          <mass value="0.008"/>
-          <inertia ixx="3.111e-7"
-                    ixy="0.0"
-                    ixz="0.0"
-                    iyy="3.600e-7"
-                    iyz="0.0"
-                    izz="3.600e-7"/>
-      </inertial>
-    </link>
-    <gazebo reference="${prefix}_roller_${suffix}_link">
-      <material>Gazebo/Black</material>
-    </gazebo>
-  </xacro:macro>
-  <!-- Half Wheel Spawn Macro -->
-  <xacro:macro name="insert_wheel" params="parent reflect prefix suffix">
-    <joint name="${prefix}_wheel${suffix}_joint" type="fixed">
-      <origin xyz="0.0 0.0 ${reflect * inter_wheel_gap/2}" rpy="0.0 0.0 ${suffix * 2*pi/28}"/>
-      <parent link="${parent}"/>
-      <child link="${prefix}_wheel${suffix}_link"/>
-    </joint>
-    <link name="${prefix}_wheel${suffix}_link">
-      <visual>
-        <origin rpy="${pi/2} 0.0 ${2*pi/28}"/>
-        <geometry>
-          <mesh filename="file://$(find omni_bot_description)/description/meshes/omni_wheel_plate.stl"/>
-        </geometry>
-        <material name="gray">
-          <color rgba="0.5 0.5 0.5 1.0"/>
-        </material>
-      </visual>
-      <!-- <collision>
-                <origin rpy="${pi/2} 0.0 ${2*pi/28}"/>
-                <geometry>
-                    <mesh filename="file://$(find omni_bot_description)/description/meshes/omni_wheel_plate.stl"/>
-                </geometry>
-      </collision> -->
-      <inertial>
-        <origin rpy="${pi/2} 0.0 ${2*pi/28}"/>
-        <mass value="0.21"/>
-        <inertia ixx="2.746e-4"
-                  ixy="0.0"
-                  ixz="0.0"
-                  iyy="0.001"
-                  iyz="0.0"
-                  izz="2.746e-4"/>
-      </inertial>
-    </link>
-    <gazebo reference="${prefix}_wheel${suffix}_link">
-      <material>Gazebo/Gray</material>
-    </gazebo>
-    <xacro:insert_roller parent="${prefix}_wheel${suffix}_link" theta="0" prefix="${prefix}_wheel${suffix}" suffix="1"/>
-    <xacro:insert_roller parent="${prefix}_wheel${suffix}_link" theta="${pi/7}" prefix="${prefix}_wheel${suffix}" suffix="2"/>
-    <xacro:insert_roller parent="${prefix}_wheel${suffix}_link" theta="${2*pi/7}" prefix="${prefix}_wheel${suffix}" suffix="3"/>
-    <xacro:insert_roller parent="${prefix}_wheel${suffix}_link" theta="${3*pi/7}" prefix="${prefix}_wheel${suffix}" suffix="4"/>
-    <xacro:insert_roller parent="${prefix}_wheel${suffix}_link" theta="${4*pi/7}" prefix="${prefix}_wheel${suffix}" suffix="5"/>
-    <xacro:insert_roller parent="${prefix}_wheel${suffix}_link" theta="${5*pi/7}" prefix="${prefix}_wheel${suffix}" suffix="6"/>
-    <xacro:insert_roller parent="${prefix}_wheel${suffix}_link" theta="${6*pi/7}" prefix="${prefix}_wheel${suffix}" suffix="7"/>
-    <xacro:insert_roller parent="${prefix}_wheel${suffix}_link" theta="${pi}" prefix="${prefix}_wheel${suffix}" suffix="8"/>
-    <xacro:insert_roller parent="${prefix}_wheel${suffix}_link" theta="${8*pi/7}" prefix="${prefix}_wheel${suffix}" suffix="9"/>
-    <xacro:insert_roller parent="${prefix}_wheel${suffix}_link" theta="${9*pi/7}" prefix="${prefix}_wheel${suffix}" suffix="10"/>
-    <xacro:insert_roller parent="${prefix}_wheel${suffix}_link" theta="${10*pi/7}" prefix="${prefix}_wheel${suffix}" suffix="11"/>
-    <xacro:insert_roller parent="${prefix}_wheel${suffix}_link" theta="${11*pi/7}" prefix="${prefix}_wheel${suffix}" suffix="12"/>
-    <xacro:insert_roller parent="${prefix}_wheel${suffix}_link" theta="${12*pi/7}" prefix="${prefix}_wheel${suffix}" suffix="13"/>
-    <xacro:insert_roller parent="${prefix}_wheel${suffix}_link" theta="${13*pi/7}" prefix="${prefix}_wheel${suffix}" suffix="14"/>
-  </xacro:macro>
   <!-- Wheel Spawn Macro -->
   <xacro:macro name="wheel" params="pos parent *origin">
@@ -103,4 +10,14 @@
     </joint>
     <link name="${pos}_wheel_link">
+      <visual>
+        <origin rpy="${pi/2} 0.0 0.0"/>
+        <geometry>
+          <mesh filename="file://$(find omni_bot_description)/description/meshes/omni_wheel_152mm.stl" />
+          <!-- <mesh filename="meshes/omni_wheel_152mm.stl" /> -->
+        </geometry>
+        <material name="dark_gray">
+          <color rgba="0.25 0.25 0.25 1.0" />
+        </material>
+      </visual>
       <collision>
         <geometry>
@@ -109,6 +26,4 @@
       </collision>
     </link>
-    <xacro:insert_wheel parent="${pos}_wheel_link" reflect="-1" prefix="${pos}" suffix="1" />
-    <xacro:insert_wheel parent="${pos}_wheel_link" reflect="1" prefix="${pos}" suffix="2" />
   </xacro:macro>
   <!-- Encoder Wheel Spawn Macro -->
@@ -125,4 +40,5 @@
         <geometry>
           <mesh filename="file://$(find omni_bot_description)/description/meshes/omni_wheel_152mm.stl" scale="${scale} ${scale} ${scale}"/>
+          <!-- <mesh filename="meshes/omni_wheel_152mm.stl" scale="${scale} ${scale} ${scale}"/> -->
         </geometry>
         <material name="light_gray">
@@ -132,5 +48,5 @@
       <collision>
         <geometry>
-          <cylinder radius="0.073" length="0.03"/>  <!-- Experimental values -->
+          <cylinder radius="${0.073 * scale}" length="${0.03 * scale}"/>  <!-- Experimental values -->
         </geometry>
       </collision>

Commit message: Edited xacro for further simplification and added a new map.

File: omni_bot_description/description/bot.xacro (robot description, xacro)
@@ -31,5 +31,5 @@
   <link name="body_link">
     <visual>
-      <origin xyz="0.0 -${base_height/3} ${base_clearance - chassis_offset}" rpy="0.0 0.0 ${pi/6}" />
+      <origin xyz="0.0 0.0 ${base_clearance - chassis_offset}" rpy="0.0 0.0 0.0" />
       <geometry>
         <mesh filename="file://$(find omni_bot_description)/description/meshes/chassis.stl" />
@@ -41,5 +41,5 @@
     </visual>
     <collision>
-      <origin xyz="0.0 -${base_height/3} ${base_clearance - chassis_offset}" rpy="0.0 0.0 ${pi/6}" />
+      <origin xyz="0.0 0.0 ${base_clearance - chassis_offset}" rpy="0.0 0.0 0.0" />
       <geometry>
         <mesh filename="file://$(find omni_bot_description)/description/meshes/chassis.stl" />
@@ -63,5 +63,5 @@
   </gazebo>
   <!-- Wheels -->
-  <xacro:wheel pos="front" parent="base_link">
+  <!-- <xacro:wheel pos="front" parent="base_link">
     <origin
       xyz="0.0 ${2 * base_height / 3 - (1.732 * corner_side_length / 2) - (rod_width / 2) - shaft_length} ${wheel_radius}"
@@ -77,5 +77,5 @@
       xyz="${((2 * base_height / 3) - (1.732 * corner_side_length / 2) - (rod_width / 2) - shaft_length)* cos(pi/6)} -${((2 * base_height / 3) - (1.732 * corner_side_length / 2) - (rod_width / 2) - shaft_length) * sin(pi/6)} ${wheel_radius}"
       rpy="${pi/2} 0.0 -${pi/6 + pi/2}" />
-  </xacro:wheel>
+  </xacro:wheel> -->
   <!-- Encoders -->
   <xacro:encoder pos="X" parent="base_link" scale="${encoder_scale}">
@@ -113,10 +113,10 @@
     <parent link="base_footprint" />
     <child link="lidar_link" />
-    <origin xyz="0.0 0.0 0.15" rpy="0.0 0.0 ${pi}" />
+    <origin xyz="0.0 0.0 0.23" rpy="0.0 0.0 ${-pi/2}" />
   </joint>
   <link name="lidar_link">
     <visual>
       <geometry>
-        <mesh filename="file://$(find omni_bot_description)/description/meshes/Scanner.stl" />
+        <!-- <mesh filename="file://$(find omni_bot_description)/description/meshes/Scanner.stl" /> -->
         <!-- <mesh filename="meshes/Scanner.stl" /> -->
       </geometry>
@@ -127,5 +127,5 @@
     <collision>
       <geometry>
-        <mesh filename="file://$(find omni_bot_description)/description/meshes/Scanner.stl" />
+        <!-- <mesh filename="file://$(find omni_bot_description)/description/meshes/Scanner.stl" /> -->
         <!-- <mesh filename="meshes/Scanner.stl" /> -->
       </geometry>

Commit message: Yet another overhaul for successful navigation and mapping (It's done!)

File: omni_bot_description/description/bot.xacro (robot description, xacro)
@@ -17,8 +17,4 @@
   <xacro:property name="base_height" value="${1.732 * base_side_length / 2}" /> <!-- m -->
   <!-- Base Link -->
-  <joint name="base_joint" type="fixed">
-    <parent link="base_link" />
-    <child link="body_link" />
-  </joint>
   <link name="base_link" />
   <!-- Base Footprint (Required by some controllers) -->
@@ -29,7 +25,12 @@
   <link name="base_footprint" />
   <!-- Base -->
+  <joint name="base_joint" type="fixed">
+    <parent link="base_link" />
+    <child link="body_link" />
+    <origin xyz="0.0 0.0 ${base_clearance - chassis_offset}" />
+  </joint>
   <link name="body_link">
     <visual>
-      <origin xyz="0.0 0.0 ${base_clearance - chassis_offset}" rpy="0.0 0.0 0.0" />
+      <origin rpy="0.0 0.0 ${-pi/2}"/>
       <geometry>
         <mesh filename="file://$(find omni_bot_description)/description/meshes/chassis.stl" />
@@ -41,5 +42,5 @@
     </visual>
     <collision>
-      <origin xyz="0.0 0.0 ${base_clearance - chassis_offset}" rpy="0.0 0.0 0.0" />
+      <origin rpy="0.0 0.0 ${-pi/2}" />
       <geometry>
         <mesh filename="file://$(find omni_bot_description)/description/meshes/chassis.stl" />
@@ -48,6 +49,4 @@
     </collision>
     <inertial>
-      <!-- <origin xyz="0.0 ${-base_height/3} ${base_clearance}" rpy="0.0 0.0 ${pi/6}"/> -->
-      <origin xyz="0.0 0.0 ${base_clearance}" rpy="0.0 0.0 0.0" />
       <mass value="${base_mass}" />
       <inertia ixx="0.1798003"
@@ -65,28 +64,33 @@
   <!-- <xacro:wheel pos="front" parent="base_link">
     <origin
-      xyz="0.0 ${2 * base_height / 3 - (1.732 * corner_side_length / 2) - (rod_width / 2) - shaft_length} ${wheel_radius}"
+      xyz="0.0 ${2 * base_height / 3 - (1.732 * corner_side_length / 2) - (rod_width / 2) - shaft_length}
+  ${wheel_radius}"
       rpy="${pi/2} 0.0 0.0" />
   </xacro:wheel>
   <xacro:wheel pos="left" parent="base_link">
     <origin
-      xyz="-${((2 * base_height / 3) - (1.732 * corner_side_length / 2) - (rod_width / 2) - shaft_length)* cos(pi/6)} -${((2 * base_height / 3) - (1.732 * corner_side_length / 2) - (rod_width / 2) - shaft_length) * sin(pi/6)} ${wheel_radius}"
+      xyz="-${((2 * base_height / 3) - (1.732 * corner_side_length / 2) - (rod_width / 2) -
+  shaft_length)* cos(pi/6)} -${((2 * base_height / 3) - (1.732 * corner_side_length / 2) -
+  (rod_width / 2) - shaft_length) * sin(pi/6)} ${wheel_radius}"
       rpy="${pi/2} 0.0 ${pi/6 + pi/2}" />
   </xacro:wheel>
   <xacro:wheel pos="right" parent="base_link">
     <origin
-      xyz="${((2 * base_height / 3) - (1.732 * corner_side_length / 2) - (rod_width / 2) - shaft_length)* cos(pi/6)} -${((2 * base_height / 3) - (1.732 * corner_side_length / 2) - (rod_width / 2) - shaft_length) * sin(pi/6)} ${wheel_radius}"
+      xyz="${((2 * base_height / 3) - (1.732 * corner_side_length / 2) - (rod_width / 2) - shaft_length)*
+  cos(pi/6)} -${((2 * base_height / 3) - (1.732 * corner_side_length / 2) - (rod_width / 2) -
+  shaft_length) * sin(pi/6)} ${wheel_radius}"
       rpy="${pi/2} 0.0 -${pi/6 + pi/2}" />
   </xacro:wheel> -->
   <!-- Encoders -->
-  <xacro:encoder pos="X" parent="base_link" scale="${encoder_scale}">
-    <origin xyz="0.0 0.08 ${encoder_radius}" rpy="-${pi/2} 0.0 0.0" />  <!-- 0.09 is experimental
+  <xacro:encoder pos="X" parent="base_footprint" scale="${encoder_scale}">
+    <origin xyz="0.08 0.0 ${encoder_radius}" rpy="${-pi/2} 0.0 ${-pi/2}" />  <!-- 0.09 is experimental
     value -->
   </xacro:encoder>
-  <xacro:encoder pos="Y" parent="base_link" scale="${encoder_scale}">
-    <origin xyz="-0.04 -0.04 ${encoder_radius}" rpy="0.0 -${pi/2} 0.0" /> <!-- 0.042 and 0.03 are
+  <xacro:encoder pos="Y" parent="base_footprint" scale="${encoder_scale}">
+    <origin xyz="-0.04 0.04 ${encoder_radius}" rpy="0.0 ${-pi/2} ${-pi/2}" /> <!-- 0.042 and 0.03 are
     experimental values -->
   </xacro:encoder>
   <!-- IMU -->
-  <joint name="imu_joint" type="fixed">
+  <!-- <joint name="imu_joint" type="fixed">
     <parent link="base_footprint" />
     <child link="imu_link" />
@@ -96,7 +100,8 @@
     <visual>
       <geometry>
-        <mesh filename="file://$(find omni_bot_description)/description/meshes/MPU_6050.stl" scale="0.001 0.001 0.001"/>
+        <mesh filename="file://$(find omni_bot_description)/description/meshes/MPU_6050.stl"
+          scale="0.001 0.001 0.001" /> -->
         <!-- <mesh filename="meshes/MPU_6050.stl" scale="0.001 0.001 0.001"/> -->
-      </geometry>
+      <!-- </geometry>
       <material name="dark_gray">
         <color rgba="0.25 0.25 0.25 1.0" />
@@ -105,18 +110,19 @@
     <collision>
       <geometry>
-        <box size="0.02 0.015 0.003"/>
+        <box size="0.02 0.015 0.003" />
       </geometry>
     </collision>
-  </link>
+  </link> -->
   <!-- Lidar -->
   <joint name="lidar_joint" type="fixed">
     <parent link="base_footprint" />
     <child link="lidar_link" />
-    <origin xyz="0.0 0.0 0.23" rpy="0.0 0.0 ${-pi/2}" />
+    <origin xyz="0.0 0.0 0.235" rpy="0.0 0.0 ${pi}" />
   </joint>
   <link name="lidar_link">
     <visual>
+      <origin xyz="0.0 0.0 -0.095"/>
       <geometry>
-        <!-- <mesh filename="file://$(find omni_bot_description)/description/meshes/Scanner.stl" /> -->
+        <mesh filename="file://$(find omni_bot_description)/description/meshes/Scanner.stl" />
         <!-- <mesh filename="meshes/Scanner.stl" /> -->
       </geometry>
@@ -127,5 +133,5 @@
     <collision>
       <geometry>
-        <!-- <mesh filename="file://$(find omni_bot_description)/description/meshes/Scanner.stl" /> -->
+        <mesh filename="file://$(find omni_bot_description)/description/meshes/Scanner.stl" />
         <!-- <mesh filename="meshes/Scanner.stl" /> -->
       </geometry>
