Commit message: Small changes to allow for GUIs (glitchy though), and minor changes (untested) for stl recognition by RViz.

File: omni_bot_description/description/bot.urdf.xacro (robot description, xacro)
@@ -20,5 +20,5 @@
       <origin xyz="-${base_side_length*sqrt(3)/6} 0.0 -${base_width/1.5}" rpy="0.0 0.0 ${-pi/3}" />
       <geometry>
-        <mesh filename="stl/chassis.stl" />
+        <mesh filename="package://omni_bot_description/description/stl/chassis.stl" />
       </geometry>
     </visual>

File: omni_bot_description/description/wheels.xacro (robot description, xacro)
@@ -38,5 +38,5 @@
         <origin xyz="0 0 0" rpy="${pi/2} 0 0" />
         <geometry>
-          <mesh filename="stl/omni_wheel_plate.stl" />
+          <mesh filename="package://omni_bot_description/description/stl/omni_wheel_plate.stl" />
         </geometry>
       </visual>
@@ -73,5 +73,5 @@
         <origin xyz="0 0 0" rpy="0 ${pi/2} 0" />
         <geometry>
-          <mesh filename="stl/omni_wheel_roller.stl" />
+          <mesh filename="package://omni_bot_description/description/stl/omni_wheel_roller.stl" />
         </geometry>
       </visual>

Commit message: - Updated devcontainer contents for GitSSH & additional ROS2 pkgs. - Setup optional script for SSH issues. - Modified URDFs for color in RViz.

File: omni_bot_description/description/bot.urdf.xacro (robot description, xacro)
@@ -22,4 +22,7 @@
         <mesh filename="package://omni_bot_description/description/stl/chassis.stl" />
       </geometry>
+      <material name="light_gray">
+        <color rgba="0.75 0.75 0.75 1.0" />
+      </material>
     </visual>
   </link>

File: omni_bot_description/description/wheels.xacro (robot description, xacro)
@@ -40,4 +40,7 @@
           <mesh filename="package://omni_bot_description/description/stl/omni_wheel_plate.stl" />
         </geometry>
+        <material name="gray">
+          <color rgba="0.5 0.5 0.5 1.0" />
+        </material>
       </visual>
     </link>
@@ -75,4 +78,7 @@
           <mesh filename="package://omni_bot_description/description/stl/omni_wheel_roller.stl" />
         </geometry>
+        <material name="black">
+          <color rgba="0.1 0.1 0.1 1.0" />
+        </material>
       </visual>
     </link>
