Commit message: Modified for 2 models: rviz and gz. All info on activating both on `URDF_Visuals.md`.

File: omni_bot_description/description/rviz_bot.urdf.xacro (robot description, xacro)
@@ -1,4 +1,4 @@
 <?xml version="1.0"?>
-<robot xmlns:xacro="http://www.ros.org/wiki/xacro" name="Omni-Bot">
+<robot xmlns:xacro="http://www.ros.org/wiki/xacro" name="rviz_Omni-Bot">
   <!--           Includes            -->
   <xacro:include filename="wheels.xacro" />
@@ -27,6 +27,12 @@
     </visual>
   </link>
-  <xacro:wheel i="0" parent="base_link" />
-  <xacro:wheel i="1" parent="base_link" />
-  <xacro:wheel i="2" parent="base_link" />
+  <xacro:wheel_preset i="0" parent="base_link" />
+  <xacro:wheel_preset i="1" parent="base_link" />
+  <xacro:wheel_preset i="2" parent="base_link" />
+  <xacro:encoder_preset i="X" parent="base_footprint">
+    <origin xyz="0.08 0.0 ${encoder_radius}" rpy="${-pi/2} 0.0 ${-pi/2}" />
+  </xacro:encoder_preset>
+  <xacro:encoder_preset i="Y" parent="base_footprint">
+    <origin xyz="-0.04 0.04 ${encoder_radius}" rpy="0.0 ${-pi/2} ${-pi/2}" />
+  </xacro:encoder_preset>
 </robot>

File: omni_bot_description/description/wheels.xacro (robot description, xacro)
@@ -8,4 +8,6 @@
   <!-- <xacro:property name="roller_width" value="0.018" /> -->
   <xacro:property name="wheel_radius" value="${plate_radius + roller_radius}" />
+  <xacro:property name="encoder_radius" value="0.05" />
+  <!--      Wheel macro       -->
   <xacro:macro name="wheel" params="i parent">
     <!--     Get wheel position      -->
@@ -27,5 +29,5 @@
     <xacro:plate i="1" parent="wheel_${i}" />
   </xacro:macro>
-  <xacro:macro name="plate" params="i parent">
+  <xacro:macro name="plate" params="i parent scale=1">
     <!--     Get plate position      -->
     <joint name="${parent}_plate_joint_${i}" type="fixed">
@@ -38,5 +40,5 @@
         <origin xyz="0 0 0" rpy="${pi/2} 0 0" />
         <geometry>
-          <mesh filename="package://omni_bot_description/description/stl/omni_wheel_plate.stl" />
+          <mesh filename="package://omni_bot_description/description/stl/omni_wheel_plate.stl" scale="${scale} ${scale} ${scale}" />
         </geometry>
         <material name="gray">
@@ -46,24 +48,24 @@
     </link>
     <!--   Add rollers to plate    -->
-    <xacro:roller i="0" parent="${parent}_plate_${i}" />
-    <xacro:roller i="1" parent="${parent}_plate_${i}" />
-    <xacro:roller i="2" parent="${parent}_plate_${i}" />
-    <xacro:roller i="3" parent="${parent}_plate_${i}" />
-    <xacro:roller i="4" parent="${parent}_plate_${i}" />
-    <xacro:roller i="5" parent="${parent}_plate_${i}" />
-    <xacro:roller i="6" parent="${parent}_plate_${i}" />
-    <xacro:roller i="7" parent="${parent}_plate_${i}" />
-    <xacro:roller i="8" parent="${parent}_plate_${i}" />
-    <xacro:roller i="9" parent="${parent}_plate_${i}" />
-    <xacro:roller i="10" parent="${parent}_plate_${i}" />
-    <xacro:roller i="11" parent="${parent}_plate_${i}" />
-    <xacro:roller i="12" parent="${parent}_plate_${i}" />
-    <xacro:roller i="13" parent="${parent}_plate_${i}" />
+    <xacro:roller i="0" parent="${parent}_plate_${i}" scale="${scale}" />
+    <xacro:roller i="1" parent="${parent}_plate_${i}" scale="${scale}" />
+    <xacro:roller i="2" parent="${parent}_plate_${i}" scale="${scale}" />
+    <xacro:roller i="3" parent="${parent}_plate_${i}" scale="${scale}" />
+    <xacro:roller i="4" parent="${parent}_plate_${i}" scale="${scale}" />
+    <xacro:roller i="5" parent="${parent}_plate_${i}" scale="${scale}" />
+    <xacro:roller i="6" parent="${parent}_plate_${i}" scale="${scale}" />
+    <xacro:roller i="7" parent="${parent}_plate_${i}" scale="${scale}" />
+    <xacro:roller i="8" parent="${parent}_plate_${i}" scale="${scale}" />
+    <xacro:roller i="9" parent="${parent}_plate_${i}" scale="${scale}" />
+    <xacro:roller i="10" parent="${parent}_plate_${i}" scale="${scale}" />
+    <xacro:roller i="11" parent="${parent}_plate_${i}" scale="${scale}" />
+    <xacro:roller i="12" parent="${parent}_plate_${i}" scale="${scale}" />
+    <xacro:roller i="13" parent="${parent}_plate_${i}" scale="${scale}" />
   </xacro:macro>
-  <xacro:macro name="roller" params="i parent">
+  <xacro:macro name="roller" params="i parent scale=1">
     <!--     Get roller position      -->
     <xacro:property name="angle" value="${i * pi/7 + pi/14}" />
-    <xacro:property name="x" value="${plate_radius * cos(angle)}" />
-    <xacro:property name="y" value="${plate_radius * sin(angle)}" />
+    <xacro:property name="x" value="${plate_radius * cos(angle) * scale}" />
+    <xacro:property name="y" value="${plate_radius * sin(angle) * scale}" />
     <joint name="${parent}_roller_joint_${i}" type="continuous">
       <parent link="${parent}" />
@@ -76,5 +78,5 @@
         <origin xyz="0 0 0" rpy="0 ${pi/2} 0" />
         <geometry>
-          <mesh filename="package://omni_bot_description/description/stl/omni_wheel_roller.stl" />
+          <mesh filename="package://omni_bot_description/description/stl/omni_wheel_roller.stl" scale="${scale} ${scale} ${scale}" />
         </geometry>
         <material name="black">
@@ -84,5 +86,68 @@
     </link>
   </xacro:macro>
-  <!--             test              -->
+  <!--        Encoder Wheels        -->
+  <xacro:macro name="encoder" params="i parent *origin">
+    <xacro:property name="encoder_scale" value="${100/152}" />
+    <joint name="encoder_joint_${i}" type="continuous">
+      <parent link="${parent}" />
+      <child link="encoder_${i}" />
+      <xacro:insert_block name="origin" />
+      <axis xyz="0 0 1" />
+      <!-- <limit lower="0.0" upper="0.0" effort="0.0" velocity="0.0"/> -->
+      <!-- <dynamics damping="0.1" friction="0.1" /> -->
+    </joint>
+    <link name="encoder_${i}">
+      <!-- A simple collision geometry -->
+    </link>
+    <xacro:plate i="0" parent="encoder_${i}" scale="${encoder_scale}"/>
+  </xacro:macro>
+  <!--        Preset Wheels          -->
+  <xacro:macro name="wheel_preset" params="i parent">
+    <!--     Get wheel position      -->
+    <xacro:property name="angle" value="${i * 2 * pi/3}" />
+    <xacro:property name="x" value="${(bot_radius + wheel_offset) * cos(angle)}" />
+    <xacro:property name="y" value="${(bot_radius + wheel_offset) * sin(angle)}" />
+    <joint name="wheel_joint_${i}" type="fixed">
+      <parent link="${parent}" />
+      <child link="wheel_${i}" />
+      <origin xyz="${x} ${y} 0" rpy="0 ${pi/2} ${angle}" />
+      <axis xyz="0 0 1" />
+    </joint>
+    <link name="wheel_${i}">
+      <visual>
+        <origin xyz="0.0 0.0 0.0" rpy="${pi/2} 0.0 0.0"/>
+        <geometry>
+          <mesh filename="package://omni_bot_description/description/stl/omni_wheel_152mm.stl" />
+        </geometry>
+        <material name="gray">
+          <color rgba="0.5 0.5 0.5 1.0" />
+        </material>
+      </visual>
+    </link>
+  </xacro:macro>
+  <!--        Encoder Preset Wheels        -->
+  <xacro:macro name="encoder_preset" params="i parent *origin">
+    <xacro:property name="encoder_scale" value="${100/152}" />
+    <joint name="encoder_joint_${i}" type="continuous">
+      <parent link="${parent}" />
+      <child link="encoder_${i}" />
+      <xacro:insert_block name="origin" />
+      <axis xyz="0 0 1" />
+      <!-- <limit lower="0.0" upper="0.0" effort="0.0" velocity="0.0"/> -->
+      <!-- <dynamics damping="0.1" friction="0.1" /> -->
+    </joint>
+    <link name="encoder_${i}">
+      <visual>
+        <origin xyz="0.0 0.0 0.0" rpy="${pi/2} 0.0 0.0"/>
+        <geometry>
+          <mesh filename="package://omni_bot_description/description/stl/omni_wheel_152mm.stl" scale="${encoder_scale} ${encoder_scale} ${encoder_scale}"/>
+        </geometry>
+        <material name="black">
+          <color rgba="0.1 0.1 0.1 1.0" />
+        </material>
+      </visual>
+    </link>
+  </xacro:macro>
+  <!--             test(wheels)              -->
   <!-- <xacro:property name="bot_radius" value="0.1" />
   <xacro:property name="wheel_offset" value="0.02" />
@@ -90,5 +155,5 @@
     <visual>
       <geometry>
-        <cylinder radius="${bot_radius}" length="0.1" />
+        <cylinder radius="${bot_radius}" length="0.05" />
       </geometry>
     </visual>
@@ -96,4 +161,29 @@
   <xacro:wheel i="0" parent="base_link" />
   <xacro:wheel i="1" parent="base_link" />
-  <xacro:wheel i="2" parent="base_link" /> -->
+  <xacro:wheel i="2" parent="base_link" />
+  <xacro:encoder i="X" parent="base_link">
+    <origin xyz="0.0 0.0 0.0" rpy="${pi/2} 0.0 0.0" />
+  </xacro:encoder>
+  <xacro:encoder i="Y" parent="base_link">
+    <origin xyz="0.0 0.0 0.0" rpy="0.0 ${pi/2} 0.0" />
+  </xacro:encoder> -->
+  <!--          test(preset)           -->
+  <!-- <xacro:property name="bot_radius" value="0.1" />
+  <xacro:property name="wheel_offset" value="0.02" />
+  <link name="base_link">
+    <visual>
+      <geometry>
+        <cylinder radius="${bot_radius}" length="0.05" />
+      </geometry>
+    </visual>
+  </link>
+  <xacro:wheel_preset i="0" parent="base_link" />
+  <xacro:wheel_preset i="1" parent="base_link" />
+  <xacro:wheel_preset i="2" parent="base_link" />
+  <xacro:encoder_preset i="X" parent="base_link">
+    <origin xyz="0.0 0.0 0.0" rpy="${pi/2} 0.0 0.0" />
+  </xacro:encoder_preset>
+  <xacro:encoder_preset i="Y" parent="base_link">
+    <origin xyz="0.0 0.0 0.0" rpy="0.0 ${pi/2} 0.0" />
+  </xacro:encoder_preset> -->
 </robot>
