Commit message: Separated the two models finally. Each RViz instance can only subscribe to one at a time to avoid TF conflict.

File: omni_bot_description/description/wheels.xacro (robot description, xacro)
@@ -143,6 +143,6 @@
           <mesh filename="package://omni_bot_description/description/stl/omni_wheel_152mm.stl" scale="${encoder_scale} ${encoder_scale} ${encoder_scale}"/>
         </geometry>
-        <material name="black">
-          <color rgba="0.1 0.1 0.1 1.0" />
+        <material name="dark_gray">
+          <color rgba="0.25 0.25 0.25 1.0" />
         </material>
       </visual>
