Commit message: Modified quite a few files to implement co-existence of both models. Ready for teleop!

File: omni_bot_description/description/gz_bot.urdf.xacro (robot description, xacro)
@@ -1,6 +1,7 @@
 <?xml version="1.0"?>
-<robot xmlns:xacro="http://www.ros.org/wiki/xacro" name="Gz_Omni-Bot">
+<robot xmlns:xacro="http://www.ros.org/wiki/xacro" name="Omni-Bot">
   <!--           Includes            -->
   <xacro:include filename="wheels.xacro" />
+  <xacro:include filename="gazebo.xacro" />
   <!--      Parameters (in SI)       -->
   <xacro:property name="base_side_length" value="1.05" />
@@ -23,7 +24,26 @@
       </geometry>
       <material name="light_gray">
-        <color rgba="0.75 0.75 0.75 1.0" />
+          <color rgba="0.75 0.75 0.75 1.0" />
+          <ambient>0.75 0.75 0.75 1</ambient>
+          <diffuse>0.75 0.75 0.75 1</diffuse>
+          <specular>0.3 0.3 0.3 1</specular>
       </material>
     </visual>
+    <collision>
+      <origin xyz="-${base_side_length*sqrt(3)/6} 0.0 -${base_width/1.5}" rpy="0.0 0.0 ${-pi/3}" />
+      <geometry>
+        <mesh filename="package://omni_bot_description/description/stl/chassis.stl" />
+      </geometry>
+    </collision>
+    <inertial>
+      <origin xyz="0.035 0.0 0.0" rpy="0.0 0.0 ${pi/6}" />
+      <mass value="${base_mass}" />
+      <inertia ixx="0.1798003"
+        ixy="0.0024346"
+        ixz="-0.0001306"
+        iyy="0.1827598"
+        iyz="-0.0002425"
+        izz="0.3538762" />
+    </inertial>
   </link>
   <xacro:wheel i="0" parent="base_link" />
@@ -31,33 +51,41 @@
   <xacro:wheel i="2" parent="base_link" />
   <!-- Spring Joints -->
+  <joint name="spring_joint_Y" type="prismatic">
+    <parent link="base_footprint" />
+    <child link="spring_link_Y" />
+    <axis xyz="0 -1 0" />
+    <origin xyz="0.08 0.0 ${encoder_radius}" rpy="${-pi/2} 0.0 ${-pi/2}" />
+    <limit lower="-0.075" upper="0.025" velocity="0.1" effort="50.0" />
+  </joint>
+  <link name="spring_link_Y">
+    <inertial>
+        <mass value="0.2"/>
+        <inertia ixx="0.000083"
+          ixy="0.0"
+          ixz="0.0"
+          iyy="0.000083"
+          iyz="0.0"
+          izz="0.000008"/>
+    </inertial>
+  </link>
   <joint name="spring_joint_X" type="prismatic">
     <parent link="base_footprint" />
     <child link="spring_link_X" />
-    <axis xyz="0 0 1" />
+    <origin xyz="-0.04 0.04 ${encoder_radius}" rpy="0.0 ${-pi/2} ${-pi/2}" />
+    <axis xyz="1 0 0" />
     <limit lower="-0.075" upper="0.025" velocity="0.1" effort="50.0" />
   </joint>
   <link name="spring_link_X">
     <inertial>
-      <mass value="0.2"/>
-      <inertia ixx="0.000083" ixy="0.0" ixz="0.0" iyy="0.000083" iyz="0.0" izz="0.000008"/>
+        <mass value="0.2"/>
+        <inertia ixx="0.000083"
+          ixy="0.0"
+          ixz="0.0"
+          iyy="0.000083"
+          iyz="0.0"
+          izz="0.000008"/>
     </inertial>
   </link>
-  <joint name="spring_joint_Y" type="prismatic">
-    <parent link="base_footprint" />
-    <child link="spring_link_Y" />
-    <axis xyz="0 0 1" />
-    <limit lower="-0.075" upper="0.025" velocity="0.1" effort="50.0" />
-  </joint>
-  <link name="spring_link_Y">
-    <inertial>
-      <mass value="0.2"/>
-      <inertia ixx="0.000083" ixy="0.0" ixz="0.0" iyy="0.000083" iyz="0.0" izz="0.000008"/>
-    </inertial>
-  </link>
-  <xacro:encoder i="X" parent="spring_link_X">
-    <origin xyz="0.08 0.0 ${encoder_radius}" rpy="${-pi/2} 0.0 ${-pi/2}" />
-  </xacro:encoder>
-  <xacro:encoder i="Y" parent="spring_link_Y">
-    <origin xyz="-0.04 0.04 ${encoder_radius}" rpy="0.0 ${-pi/2} ${-pi/2}" />
-  </xacro:encoder>
+  <xacro:encoder i="X" parent="spring_link_X" />
+  <xacro:encoder i="Y" parent="spring_link_Y" />
 </robot>

File: omni_bot_description/description/rviz_bot.urdf.xacro (robot description, xacro)
@@ -26,4 +26,15 @@
       </material>
     </visual>
+    <collision>
+      <origin xyz="-${base_side_length*sqrt(3)/6} 0.0 -${base_width/1.5}" rpy="0.0 0.0 ${-pi/3}" />
+      <geometry>
+        <mesh filename="package://omni_bot_description/description/stl/chassis.stl" />
+      </geometry>
+    </collision>
+    <inertial>
+      <origin xyz="0.0 0.0 0.0" />
+      <mass value="${base_mass}" />
+      <inertia ixx="0.1798003" ixy="0.0024346" ixz="-0.0001306" iyy="0.1827598" iyz="-0.0002425" izz="0.3538762" />
+    </inertial>
   </link>
   <xacro:wheel_preset i="0" parent="base_link" />
@@ -31,8 +42,8 @@
   <xacro:wheel_preset i="2" parent="base_link" />
   <xacro:encoder_preset i="X" parent="base_footprint">
+    <origin xyz="-0.04 0.04 ${encoder_radius}" rpy="0.0 ${-pi/2} ${-pi/2}" />
+  </xacro:encoder_preset>
+  <xacro:encoder_preset i="Y" parent="base_footprint">
     <origin xyz="0.08 0.0 ${encoder_radius}" rpy="${-pi/2} 0.0 ${-pi/2}" />
   </xacro:encoder_preset>
-  <xacro:encoder_preset i="Y" parent="base_footprint">
-    <origin xyz="-0.04 0.04 ${encoder_radius}" rpy="0.0 ${-pi/2} ${-pi/2}" />
-  </xacro:encoder_preset>
 </robot>

File: omni_bot_description/description/wheels.xacro (robot description, xacro)
@@ -5,6 +5,7 @@
   <xacro:property name="plate_radius" value="0.0675" />
   <xacro:property name="plate_gap" value="0.02" />
+  <xacro:property name="roller_mass" value="0.008" />
   <xacro:property name="roller_radius" value="0.0095" />
-  <!-- <xacro:property name="roller_width" value="0.018" /> -->
+  <xacro:property name="roller_length" value="0.018" />
   <xacro:property name="wheel_radius" value="${plate_radius + roller_radius}" />
   <xacro:property name="encoder_radius" value="0.05" />
@@ -20,9 +21,23 @@
       <origin xyz="${x} ${y} 0" rpy="0 ${pi/2} ${angle}" />
       <axis xyz="0 0 1" />
-      <!-- <limit lower="0.0" upper="0.0" effort="0.0" velocity="0.0"/> -->
-      <!-- <dynamics damping="0.1" friction="0.1" /> -->
+      <dynamics damping="25e-4" friction="1e-4"/>
     </joint>
     <link name="wheel_${i}">
       <!-- A simple collision geometry -->
+      <collision>
+        <geometry>
+          <cylinder radius="${plate_radius}" length="${plate_gap}" />
+        </geometry>
+      </collision>
+      <!-- Fake Inertial (Actual values in plate)-->
+      <inertial>
+        <mass value="1e-6" />
+        <inertia ixx="1e-9"
+          ixy="0"
+          ixz="0"
+          iyy="1e-9"
+          iyz="0"
+          izz="1e-9"/>
+      </inertial>
     </link>
     <xacro:plate i="-1" parent="wheel_${i}" />
@@ -41,7 +56,11 @@
         <geometry>
           <mesh filename="package://omni_bot_description/description/stl/omni_wheel_plate.stl" scale="${scale} ${scale} ${scale}" />
+          <!-- <cylinder radius="${plate_radius * scale}" length="${plate_gap/2}"/> -->
         </geometry>
         <material name="gray">
           <color rgba="0.5 0.5 0.5 1.0" />
+          <ambient>0.1 0.1 0.1 1</ambient>
+          <diffuse>0.2 0.2 0.2 1</diffuse>
+          <specular>0.1 0.1 0.1 1</specular>
         </material>
       </visual>
@@ -73,4 +92,5 @@
       <origin xyz="${x} ${y} 0" rpy="${pi/2} 0 ${angle}" />
       <axis xyz="0 0 1" />
+      <dynamics damping="1e-5" friction="1e-5"/>
     </joint>
     <link name="${parent}_roller_${i}">
@@ -82,23 +102,52 @@
         <material name="black">
           <color rgba="0.1 0.1 0.1 1.0" />
-        </material>
-      </visual>
+          <ambient>0.02 0.02 0.02 1</ambient>
+          <diffuse>0.05 0.05 0.05 1</diffuse>
+          <specular>0.01 0.01 0.01 1</specular>
+        </material>
+      </visual>
+      <collision>
+        <geometry>
+          <cylinder radius="${roller_radius * scale}" length="${roller_length * scale}" />
+        </geometry>
+      </collision>
+      <inertial>
+          <mass value="${roller_mass}"/>
+          <inertia ixx="3.111e-7"
+            ixy="0.0"
+            ixz="0.0"
+            iyy="3.600e-7"
+            iyz="0.0"
+            izz="3.600e-7"/>
+      </inertial>
     </link>
   </xacro:macro>
   <!--        Encoder Wheels        -->
-  <xacro:macro name="encoder" params="i parent *origin">
+  <xacro:macro name="encoder" params="i parent">
     <xacro:property name="encoder_scale" value="${100/152}" />
     <joint name="encoder_joint_${i}" type="continuous">
       <parent link="${parent}" />
       <child link="encoder_${i}" />
-      <xacro:insert_block name="origin" />
-      <axis xyz="0 0 1" />
-      <!-- <limit lower="0.0" upper="0.0" effort="0.0" velocity="0.0"/> -->
-      <!-- <dynamics damping="0.1" friction="0.1" /> -->
+      <axis xyz="0 0 1" />
     </joint>
     <link name="encoder_${i}">
       <!-- A simple collision geometry -->
-    </link>
-    <xacro:plate i="0" parent="encoder_${i}" scale="${encoder_scale}"/>
+      <collision>
+        <geometry>
+          <cylinder radius="${plate_radius * encoder_scale}" length="${plate_gap * encoder_scale}" />
+        </geometry>
+      </collision>
+      <!-- Fake Inertial (Actual values in plate)-->
+      <inertial>
+        <mass value="1e-6" />
+        <inertia ixx="1e-9"
+          ixy="0"
+          ixz="0"
+          iyy="1e-9"
+          iyz="0"
+          izz="1e-9"/>
+      </inertial>
+    </link>
+    <xacro:plate i="0" parent="encoder_${i}" scale="${encoder_scale}" />
   </xacro:macro>
   <!--        Preset Wheels          -->
@@ -116,5 +165,5 @@
     <link name="wheel_${i}">
       <visual>
-        <origin xyz="0.0 0.0 0.0" rpy="${pi/2} 0.0 0.0"/>
+        <origin xyz="0.0 0.0 0.0" rpy="${pi/2} 0.0 0.0" />
         <geometry>
           <mesh filename="package://omni_bot_description/description/stl/omni_wheel_152mm.stl" />
@@ -124,4 +173,9 @@
         </material>
       </visual>
+      <collision>
+        <geometry>
+          <cylinder radius="${wheel_radius}" length="${plate_gap + 2*roller_radius}" />
+        </geometry>
+      </collision>
     </link>
   </xacro:macro>
@@ -139,12 +193,17 @@
     <link name="encoder_${i}">
       <visual>
-        <origin xyz="0.0 0.0 0.0" rpy="${pi/2} 0.0 0.0"/>
-        <geometry>
-          <mesh filename="package://omni_bot_description/description/stl/omni_wheel_152mm.stl" scale="${encoder_scale} ${encoder_scale} ${encoder_scale}"/>
+        <origin xyz="0.0 0.0 0.0" rpy="${pi/2} 0.0 0.0" />
+        <geometry>
+          <mesh filename="package://omni_bot_description/description/stl/omni_wheel_152mm.stl" scale="${encoder_scale} ${encoder_scale} ${encoder_scale}" />
         </geometry>
         <material name="dark_gray">
-          <color rgba="0.25 0.25 0.25 1.0" />
-        </material>
-      </visual>
+          <color rgba="0.35 0.35 0.35 1.0" />
+        </material>
+      </visual>
+      <collision>
+        <geometry>
+          <cylinder radius="${wheel_radius * encoder_scale}" length="${(plate_gap + 2*roller_radius) * encoder_scale}" />
+        </geometry>
+      </collision>
     </link>
   </xacro:macro>
