Commit message: Massive changes: - New pkg for wheel speed calculation - New pkg for odometry from encoder calculation - Minor modifications to make `/robot_description` compatible with ros2_control. Possible Issues: - RViz model now has "continuous" wheels, so fake TF broadcasting is needed in HW. - Minor glitches in `/cmd_vel` topic, possibly due to duplication of Publishers.

File: omni_bot_description/description/gazebo.xacro (robot description, xacro)
@@ -1,9 +1,16 @@
 <robot xmlns:xacro="http://www.ros.org/wiki/xacro">
   <gazebo>
-    <!-- Joint States -->
+    <!-- Joint States Publisher (for encoders and other passive joints) -->
     <plugin filename="gz-sim-joint-state-publisher-system" name="gz::sim::systems::JointStatePublisher">
+      <topic>joint_states</topic>
       <joint_name>encoder_joint_X</joint_name>
       <joint_name>encoder_joint_Y</joint_name>
-      <topic>joint_states</topic>
+      <joint_name>wheel_joint_0</joint_name>
+      <joint_name>wheel_joint_1</joint_name>
+      <joint_name>wheel_joint_2</joint_name>
+    </plugin>
+    <!-- Gazebo ros2_control plugin -->
+    <plugin filename="gz_ros2_control-system" name="gz_ros2_control::GazeboSimROS2ControlPlugin">
+      <parameters>$(find omni_bot_sim)/config/omni_controller.yaml</parameters>
     </plugin>
   </gazebo>

File: omni_bot_description/description/gz_bot.urdf.xacro (robot description, xacro)
@@ -24,8 +24,8 @@
       </geometry>
       <material name="light_gray">
-          <color rgba="0.75 0.75 0.75 1.0" />
-          <ambient>0.75 0.75 0.75 1</ambient>
-          <diffuse>0.75 0.75 0.75 1</diffuse>
-          <specular>0.3 0.3 0.3 1</specular>
+        <color rgba="0.75 0.75 0.75 1.0" />
+        <ambient>0.75 0.75 0.75 1</ambient>
+        <diffuse>0.75 0.75 0.75 1</diffuse>
+        <specular>0.3 0.3 0.3 1</specular>
       </material>
     </visual>
@@ -39,10 +39,5 @@
       <origin xyz="0.035 0.0 0.0" rpy="0.0 0.0 ${pi/6}" />
       <mass value="${base_mass}" />
-      <inertia ixx="0.1798003"
-        ixy="0.0024346"
-        ixz="-0.0001306"
-        iyy="0.1827598"
-        iyz="-0.0002425"
-        izz="0.3538762" />
+      <inertia ixx="0.1798003" ixy="0.0024346" ixz="-0.0001306" iyy="0.1827598" iyz="-0.0002425" izz="0.3538762" />
     </inertial>
   </link>
@@ -60,11 +55,6 @@
   <link name="spring_link_Y">
     <inertial>
-        <mass value="0.2"/>
-        <inertia ixx="0.000083"
-          ixy="0.0"
-          ixz="0.0"
-          iyy="0.000083"
-          iyz="0.0"
-          izz="0.000008"/>
+      <mass value="0.2" />
+      <inertia ixx="0.000083" ixy="0.0" ixz="0.0" iyy="0.000083" iyz="0.0" izz="0.000008" />
     </inertial>
   </link>
@@ -78,11 +68,6 @@
   <link name="spring_link_X">
     <inertial>
-        <mass value="0.2"/>
-        <inertia ixx="0.000083"
-          ixy="0.0"
-          ixz="0.0"
-          iyy="0.000083"
-          iyz="0.0"
-          izz="0.000008"/>
+      <mass value="0.2" />
+      <inertia ixx="0.000083" ixy="0.0" ixz="0.0" iyy="0.000083" iyz="0.0" izz="0.000008" />
     </inertial>
   </link>

File: omni_bot_description/description/rviz_bot.urdf.xacro (robot description, xacro)
@@ -3,4 +3,5 @@
   <!--           Includes            -->
   <xacro:include filename="wheels.xacro" />
+  <xacro:include filename="ros2_control.xacro" />
   <!--      Parameters (in SI)       -->
   <xacro:property name="base_side_length" value="1.05" />

File: omni_bot_description/description/wheels.xacro (robot description, xacro)
@@ -21,5 +21,5 @@
       <origin xyz="${x} ${y} 0" rpy="0 ${pi/2} ${angle}" />
       <axis xyz="0 0 1" />
-      <dynamics damping="25e-4" friction="1e-4"/>
+      <dynamics damping="25e-4" friction="1e-4" />
     </joint>
     <link name="wheel_${i}">
@@ -33,10 +33,5 @@
       <inertial>
         <mass value="1e-6" />
-        <inertia ixx="1e-9"
-          ixy="0"
-          ixz="0"
-          iyy="1e-9"
-          iyz="0"
-          izz="1e-9"/>
+        <inertia ixx="1e-9" ixy="0" ixz="0" iyy="1e-9" iyz="0" izz="1e-9" />
       </inertial>
     </link>
@@ -92,5 +87,5 @@
       <origin xyz="${x} ${y} 0" rpy="${pi/2} 0 ${angle}" />
       <axis xyz="0 0 1" />
-      <dynamics damping="1e-5" friction="1e-5"/>
+      <dynamics damping="1e-5" friction="1e-5" />
     </joint>
     <link name="${parent}_roller_${i}">
@@ -113,11 +108,6 @@
       </collision>
       <inertial>
-          <mass value="${roller_mass}"/>
-          <inertia ixx="3.111e-7"
-            ixy="0.0"
-            ixz="0.0"
-            iyy="3.600e-7"
-            iyz="0.0"
-            izz="3.600e-7"/>
+        <mass value="${roller_mass}" />
+        <inertia ixx="3.111e-7" ixy="0.0" ixz="0.0" iyy="3.600e-7" iyz="0.0" izz="3.600e-7" />
       </inertial>
     </link>
@@ -141,10 +131,5 @@
       <inertial>
         <mass value="1e-6" />
-        <inertia ixx="1e-9"
-          ixy="0"
-          ixz="0"
-          iyy="1e-9"
-          iyz="0"
-          izz="1e-9"/>
+        <inertia ixx="1e-9" ixy="0" ixz="0" iyy="1e-9" iyz="0" izz="1e-9" />
       </inertial>
     </link>
@@ -157,5 +142,5 @@
     <xacro:property name="x" value="${(bot_radius + wheel_offset) * cos(angle)}" />
     <xacro:property name="y" value="${(bot_radius + wheel_offset) * sin(angle)}" />
-    <joint name="wheel_joint_${i}" type="fixed">
+    <joint name="wheel_joint_${i}" type="continuous">
       <parent link="${parent}" />
       <child link="wheel_${i}" />

Commit message: Minor (but VERY affecting) update: - IMU integration added to bot, allowing to (nearly) correctly track both position and orientation. Possible improvements: - Currently only Yaw used; can implement EKF to merge enoders w/ accel values.

File: omni_bot_description/description/gazebo.xacro (robot description, xacro)
@@ -14,4 +14,20 @@
       <parameters>$(find omni_bot_sim)/config/omni_controller.yaml</parameters>
     </plugin>
+    <!-- IMU plugin -->
+    <plugin filename="gz-sim-imu-system" name="gz::sim::systems::Imu">
+    </plugin>
+  </gazebo>
+  <!-- Ideal IMU attached to imu_link -->
+  <gazebo reference="imu_link">
+    <sensor name="imu_sensor" type="imu">
+      <always_on>1</always_on>
+      <update_rate>200</update_rate>
+      <visualize>true</visualize>
+      <topic>imu</topic>
+      <pose>0 0 0 0 0 0</pose>
+      <imu>
+        <!-- Ideal IMU: no noise configured -->
+      </imu>
+    </sensor>
   </gazebo>
 </robot>

File: omni_bot_description/description/gz_bot.urdf.xacro (robot description, xacro)
@@ -42,4 +42,30 @@
     </inertial>
   </link>
+  <!-- IMU frame placed 0.10 m above base_link origin -->
+  <joint name="imu_joint" type="fixed">
+    <parent link="base_link" />
+    <child link="imu_link" />
+    <origin xyz="0 0 0.05" rpy="0 0 0" />
+  </joint>
+  <link name="imu_link">
+    <inertial>
+      <mass value="0.01" />
+      <inertia ixx="1e-6" ixy="0" ixz="0" iyy="1e-6" iyz="0" izz="1e-6" />
+    </inertial>
+    <visual>
+      <origin xyz="0 0 0" rpy="0 0 0" />
+      <geometry>
+        <box size="0.02 0.02 0.01" />
+      </geometry>
+      <material name="blue">
+        <color rgba="0.2 0.2 0.8 0.8" />
+      </material>
+    </visual>
+    <collision>
+      <geometry>
+        <box size="0.02 0.02 0.01" />
+      </geometry>
+    </collision>
+  </link>
   <xacro:wheel i="0" parent="base_link" />
   <xacro:wheel i="1" parent="base_link" />

Commit message: Patch: LiDAR works, but need to add `LaserScan` message to RViz.

File: omni_bot_description/description/gazebo.xacro (robot description, xacro)
@@ -1,4 +1,15 @@
 <robot xmlns:xacro="http://www.ros.org/wiki/xacro">
+  <!-- Gazebo System Plugins and Sensor Configuration
+       CRITICAL: Define system plugins here for all Gazebo features (sensors, control, physics)
+       Reference: https://github.com/gazebosim/gz-sim
+  -->
   <gazebo>
+    <!-- CRITICAL: Gazebo Sensors System Plugin
+         Without this plugin, sensors (LiDAR, IMU, cameras) will NOT publish topics.
+         This plugin must be included either here (URDF/Xacro) or in the world file (but not both).
+    -->
+    <plugin filename="gz-sim-sensors-system" name="gz::sim::systems::Sensors">
+      <render_engine>ogre2</render_engine>
+    </plugin>
     <!-- Joint States Publisher (for encoders and other passive joints) -->
     <plugin filename="gz-sim-joint-state-publisher-system" name="gz::sim::systems::JointStatePublisher">
@@ -21,8 +32,8 @@
   <gazebo reference="imu_link">
     <sensor name="imu_sensor" type="imu">
-      <always_on>1</always_on>
+      <topic>imu</topic>
+      <always_on>true</always_on>
       <update_rate>200</update_rate>
       <visualize>true</visualize>
-      <topic>imu</topic>
       <pose>0 0 0 0 0 0</pose>
       <imu>
@@ -31,3 +42,46 @@
     </sensor>
   </gazebo>
+  <!-- Gazebo LiDAR Plugin Configuration for YDLiDAR G2 -->
+  <!-- CRITICAL: Gazebo plugin for GPU LiDAR -->
+  <!-- Reference: YDLidar_G2.md (Factory Fresh Plug-and-Play Specifications) -->
+  <gazebo reference="lidar_link">
+    <material>Gazebo/Black</material>
+    <!-- YDLiDAR G2 Hardware Characteristics:
+         - Field of View: 360° (full continuous rotation)
+         - Motor Speed: ~8 Hz (480 RPM)
+         - Sampling Rate: ~5000 samples/second
+         - Angular Resolution: ~0.36°
+         - Range: 0.12m to 12.0m
+         - Communication: UART via USB-TTL @ 230400 bps (plug-and-play)
+    -->
+    <!-- Type: gpu_lidar (not ray or lidar) for modern Gazebo (Harmonic/Garden) -->
+    <sensor name="lidar_sensor" type="gpu_lidar">
+      <pose>0 0 0 0 0 0</pose>
+      <visualize>true</visualize>
+      <update_rate>10</update_rate>
+      <topic>scan</topic>
+      <!-- CRITICAL: Sets the frame_id in LaserScan messages -->
+      <!-- MUST match the link name (lidar_link) for TF consistency -->
+      <!-- Without this, Gazebo auto-generates frame like robot_name/parent_link/sensor_name -->
+      <gz_frame_id>lidar_link</gz_frame_id>
+      <lidar>
+        <scan>
+          <horizontal>
+            <!-- YDLiDAR G2: 360° full rotation scanning -->
+            <!-- 1.0° resolution = 360 samples per complete rotation -->
+            <!-- Native sensor: ~0.36° angular resolution, 5000 samples/sec -->
+            <samples>360</samples>
+            <!-- Full 360° field of view: -180° to +180° -->
+            <min_angle>-3.14159</min_angle>
+            <max_angle>3.14159</max_angle>
+          </horizontal>
+        </scan>
+        <range>
+          <!-- YDLiDAR G2 Range: 0.12m to 12.0m -->
+          <min>0.12</min>
+          <max>12.0</max>
+        </range>
+      </lidar>
+    </sensor>
+  </gazebo>
 </robot>

File: omni_bot_description/description/gz_bot.urdf.xacro (robot description, xacro)
@@ -2,5 +2,8 @@
 <robot xmlns:xacro="http://www.ros.org/wiki/xacro" name="Omni-Bot">
   <!--           Includes            -->
+  <xacro:include filename="inertial_macros.xacro" />
   <xacro:include filename="wheels.xacro" />
+  <xacro:include filename="lidar.xacro" />
+  <xacro:include filename="imu.xacro" />
   <xacro:include filename="gazebo.xacro" />
   <!--      Parameters (in SI)       -->
@@ -42,30 +45,12 @@
     </inertial>
   </link>
-  <!-- IMU frame placed 0.10 m above base_link origin -->
-  <joint name="imu_joint" type="fixed">
-    <parent link="base_link" />
-    <child link="imu_link" />
-    <origin xyz="0 0 0.05" rpy="0 0 0" />
-  </joint>
-  <link name="imu_link">
-    <inertial>
-      <mass value="0.01" />
-      <inertia ixx="1e-6" ixy="0" ixz="0" iyy="1e-6" iyz="0" izz="1e-6" />
-    </inertial>
-    <visual>
-      <origin xyz="0 0 0" rpy="0 0 0" />
-      <geometry>
-        <box size="0.02 0.02 0.01" />
-      </geometry>
-      <material name="blue">
-        <color rgba="0.2 0.2 0.8 0.8" />
-      </material>
-    </visual>
-    <collision>
-      <geometry>
-        <box size="0.02 0.02 0.01" />
-      </geometry>
-    </collision>
-  </link>
+  <!-- IMU frame placed 0.148 m above base_footprint origin -->
+  <xacro:imu_mpu6050 parent="base_footprint">
+    <origin xyz="0 0 0.148" rpy="0 0 0" />
+  </xacro:imu_mpu6050>
+  <!-- LiDAR mounted 0.235m above base_footprint -->
+  <xacro:ydlidar_g2 parent="base_footprint">
+    <origin xyz="0 0 0.25" rpy="0 0 0" />
+  </xacro:ydlidar_g2>
   <xacro:wheel i="0" parent="base_link" />
   <xacro:wheel i="1" parent="base_link" />

File: omni_bot_description/description/rviz_bot.urdf.xacro (robot description, xacro)
@@ -3,4 +3,6 @@
   <!--           Includes            -->
   <xacro:include filename="wheels.xacro" />
+  <xacro:include filename="lidar.xacro" />
+  <xacro:include filename="imu.xacro" />
   <xacro:include filename="ros2_control.xacro" />
   <!--      Parameters (in SI)       -->
@@ -39,4 +41,12 @@
     </inertial>
   </link>
+  <!-- IMU frame placed 0.148 m above base_footprint origin -->
+  <xacro:imu_mpu6050 parent="base_footprint">
+    <origin xyz="0 0 0.148" rpy="0 0 0" />
+  </xacro:imu_mpu6050>
+  <!-- LiDAR mounted 0.235m above base_footprint -->
+  <xacro:ydlidar_g2 parent="base_footprint">
+    <origin xyz="0 0 0.25" rpy="0 0 0" />
+  </xacro:ydlidar_g2>
   <xacro:wheel_preset i="0" parent="base_link" />
   <xacro:wheel_preset i="1" parent="base_link" />

Commit message: Major chnages for sim parity: - Added `use_sim_time` arg to many files. - URDF parity changes; though no overall effect visible. - Updated `omni_bot_navigation` pkg to be much more smarter. - Used args like `use_sim_time` to dynamically switch between real and sim launches, and localization src selection.

File: omni_bot_description/description/gazebo.xacro (robot description, xacro)
@@ -1,17 +1,11 @@
 <robot xmlns:xacro="http://www.ros.org/wiki/xacro">
-  <!-- Gazebo System Plugins and Sensor Configuration
-       CRITICAL: Define system plugins here for all Gazebo features (sensors, control, physics)
-       Reference: https://github.com/gazebosim/gz-sim
-  -->
   <gazebo>
-    <!-- CRITICAL: Gazebo Sensors System Plugin
-         Without this plugin, sensors (LiDAR, IMU, cameras) will NOT publish topics.
-         This plugin must be included either here (URDF/Xacro) or in the world file (but not both).
-    -->
+    <!-- Sensors System Plugin (required for IMU, LIDAR, etc.) -->
     <plugin filename="gz-sim-sensors-system" name="gz::sim::systems::Sensors">
       <render_engine>ogre2</render_engine>
     </plugin>
     <!-- Joint States Publisher (for encoders and other passive joints) -->
-    <plugin filename="gz-sim-joint-state-publisher-system" name="gz::sim::systems::JointStatePublisher">
+    <plugin filename="gz-sim-joint-state-publisher-system"
+      name="gz::sim::systems::JointStatePublisher">
       <topic>joint_states</topic>
       <joint_name>encoder_joint_X</joint_name>
@@ -42,7 +36,5 @@
     </sensor>
   </gazebo>
-  <!-- Gazebo LiDAR Plugin Configuration for YDLiDAR G2 -->
-  <!-- CRITICAL: Gazebo plugin for GPU LiDAR -->
-  <!-- Reference: YDLidar_G2.md (Factory Fresh Plug-and-Play Specifications) -->
+  <!-- YDLiDAR G2 360° 2D LiDAR Sensor attached to lidar_link -->
   <gazebo reference="lidar_link">
     <material>Gazebo/Black</material>
@@ -68,9 +60,5 @@
         <scan>
           <horizontal>
-            <!-- YDLiDAR G2: 360° full rotation scanning -->
-            <!-- 1.0° resolution = 360 samples per complete rotation -->
-            <!-- Native sensor: ~0.36° angular resolution, 5000 samples/sec -->
             <samples>360</samples>
-            <!-- Full 360° field of view: -180° to +180° -->
             <min_angle>-3.14159</min_angle>
             <max_angle>3.14159</max_angle>

File: omni_bot_description/description/gz_bot.urdf.xacro (robot description, xacro)
@@ -42,5 +42,6 @@
       <origin xyz="0.035 0.0 0.0" rpy="0.0 0.0 ${pi/6}" />
       <mass value="${base_mass}" />
-      <inertia ixx="0.1798003" ixy="0.0024346" ixz="-0.0001306" iyy="0.1827598" iyz="-0.0002425" izz="0.3538762" />
+      <inertia ixx="0.1798003" ixy="0.0024346" ixz="-0.0001306" iyy="0.1827598" iyz="-0.0002425"
+        izz="0.3538762" />
     </inertial>
   </link>
@@ -51,5 +52,5 @@
   <!-- LiDAR mounted 0.235m above base_footprint -->
   <xacro:ydlidar_g2 parent="base_footprint">
-    <origin xyz="0 0 0.25" rpy="0 0 0" />
+    <origin xyz="0 0 0.25" rpy="0 0 ${2*pi}" />   <!-- Parity with Hardware -->
   </xacro:ydlidar_g2>
   <xacro:wheel i="0" parent="base_link" />

Commit message: Aim of the branch: - Ensure similarity of motor response between sim and reality. - Ensure same data type consumed by both sim and real.

File: omni_bot_description/description/gazebo.xacro (robot description, xacro)
@@ -15,7 +15,19 @@
       <joint_name>wheel_joint_2</joint_name>
     </plugin>
-    <!-- Gazebo ros2_control plugin -->
-    <plugin filename="gz_ros2_control-system" name="gz_ros2_control::GazeboSimROS2ControlPlugin">
-      <parameters>$(find omni_bot_sim)/config/omni_controller.yaml</parameters>
+    <!-- Gazebo Joint Controller (for controlling wheel joints) -->
+    <plugin filename="gz-sim-joint-controller-system" name="gz::sim::systems::JointController">
+      <topic>/omni_controller/commands/wheel_0</topic>
+      <joint_name>wheel_joint_0</joint_name>
+      <use_force_commands>true</use_force_commands>
+    </plugin>
+    <plugin filename="gz-sim-joint-controller-system" name="gz::sim::systems::JointController">
+      <topic>/omni_controller/commands/wheel_1</topic>
+      <joint_name>wheel_joint_1</joint_name>
+      <use_force_commands>true</use_force_commands>
+    </plugin>
+    <plugin filename="gz-sim-joint-controller-system" name="gz::sim::systems::JointController">
+      <topic>/omni_controller/commands/wheel_2</topic>
+      <joint_name>wheel_joint_2</joint_name>
+      <use_force_commands>true</use_force_commands>
     </plugin>
     <!-- IMU plugin -->

File: omni_bot_description/description/gz_bot.urdf.xacro (robot description, xacro)
@@ -43,5 +43,5 @@
       <mass value="${base_mass}" />
       <inertia ixx="0.1798003" ixy="0.0024346" ixz="-0.0001306" iyy="0.1827598" iyz="-0.0002425"
-        izz="0.3538762" />
+        izz="0.01" />  <!-- Tune Izz w/ real HW for correct rotation -->
     </inertial>
   </link>

File: omni_bot_description/description/rviz_bot.urdf.xacro (robot description, xacro)
@@ -5,5 +5,5 @@
   <xacro:include filename="lidar.xacro" />
   <xacro:include filename="imu.xacro" />
-  <xacro:include filename="ros2_control.xacro" />
+  <!-- <xacro:include filename="ros2_control.xacro" /> -->
   <!--      Parameters (in SI)       -->
   <xacro:property name="base_side_length" value="1.05" />
@@ -38,5 +38,6 @@
       <origin xyz="0.0 0.0 0.0" />
       <mass value="${base_mass}" />
-      <inertia ixx="0.1798003" ixy="0.0024346" ixz="-0.0001306" iyy="0.1827598" iyz="-0.0002425" izz="0.3538762" />
+      <inertia ixx="0.1798003" ixy="0.0024346" ixz="-0.0001306" iyy="0.1827598" iyz="-0.0002425"
+        izz="0.3538762" />
     </inertial>
   </link>

File: omni_bot_description/description/wheels.xacro (robot description, xacro)
@@ -10,4 +10,6 @@
   <xacro:property name="wheel_radius" value="${plate_radius + roller_radius}" />
   <xacro:property name="encoder_radius" value="0.05" />
+  <xacro:property name="wheel_damping" value="0.45" />
+  <xacro:property name="wheel_friction" value="1e-4" />
   <!--      Wheel macro       -->
   <xacro:macro name="wheel" params="i parent">
@@ -21,5 +23,5 @@
       <origin xyz="${x} ${y} 0" rpy="0 ${pi/2} ${angle}" />
       <axis xyz="0 0 1" />
-      <dynamics damping="25e-4" friction="1e-4" />
+      <dynamics damping="${wheel_damping}" friction="${wheel_friction}" />
     </joint>
     <link name="wheel_${i}">
@@ -50,5 +52,6 @@
         <origin xyz="0 0 0" rpy="${pi/2} 0 0" />
         <geometry>
-          <mesh filename="package://omni_bot_description/description/stl/omni_wheel_plate.stl" scale="${scale} ${scale} ${scale}" />
+          <mesh filename="package://omni_bot_description/description/stl/omni_wheel_plate.stl"
+            scale="${scale} ${scale} ${scale}" />
           <!-- <cylinder radius="${plate_radius * scale}" length="${plate_gap/2}"/> -->
         </geometry>
@@ -93,5 +96,6 @@
         <origin xyz="0 0 0" rpy="0 ${pi/2} 0" />
         <geometry>
-          <mesh filename="package://omni_bot_description/description/stl/omni_wheel_roller.stl" scale="${scale} ${scale} ${scale}" />
+          <mesh filename="package://omni_bot_description/description/stl/omni_wheel_roller.stl"
+            scale="${scale} ${scale} ${scale}" />
         </geometry>
         <material name="black">
@@ -180,5 +184,6 @@
         <origin xyz="0.0 0.0 0.0" rpy="${pi/2} 0.0 0.0" />
         <geometry>
-          <mesh filename="package://omni_bot_description/description/stl/omni_wheel_152mm.stl" scale="${encoder_scale} ${encoder_scale} ${encoder_scale}" />
+          <mesh filename="package://omni_bot_description/description/stl/omni_wheel_152mm.stl"
+            scale="${encoder_scale} ${encoder_scale} ${encoder_scale}" />
         </geometry>
         <material name="dark_gray">
@@ -188,5 +193,6 @@
       <collision>
         <geometry>
-          <cylinder radius="${wheel_radius * encoder_scale}" length="${(plate_gap + 2*roller_radius) * encoder_scale}" />
+          <cylinder radius="${wheel_radius * encoder_scale}"
+            length="${(plate_gap + 2*roller_radius) * encoder_scale}" />
         </geometry>
       </collision>
